File: KiCad/uSpoke.kicad_pcb (KiCad board)
At the start: 2 copper layers, 30 x 50 mm, 70 parts, among them J1 PLS-1x4, J2 Untitled, J3 PLS-1x3, J4 SMA, Q1 AO3407A, Q2 AO3400, Q3 AO3400, SW1 TL3330AF260QG, SW2 TL3330AF260QG, SW3 TL3330AF260QG, U1 SP0503BAHTG, U2 LM3671MF-3.3, U3 MCP73831T-2ACI/OT, U4 74HC4052PW, U5 STM32F103C8T6, X1 8MHz

Commit message: Main placement done
Parts:
- moved C11 101.7 mm to (97.0, 110.7), turned to 0 degrees
- moved C13 93.1 mm to (97.0, 113.5), turned to 0 degrees
- moved R4 91.8 mm to (87.0, 107.4), turned to 180 degrees
- moved C15 90.7 mm to (82.5, 116.5), turned to 180 degrees
- moved R15 90.1 mm to (97.0, 112.0), turned to 0 degrees
- moved X1 79.7 mm to (97.0, 116.3), turned to 90 degrees
- moved R18 75.1 mm to (82.5, 118.1)
- moved C8 74.9 mm to (114.3, 112.0)
- moved C10 66.8 mm to (91.7, 119.6), turned to 180 degrees
- moved C9 66.4 mm to (97.0, 119.1), turned to 180 degrees
- moved C12 59.7 mm to (84.8, 108.9), turned to 180 degrees
- moved U5 46.0 mm to (89.7, 113.2), turned to 180 degrees
- moved C19 27.0 mm to (101.8, 108.4), turned to 90 degrees
- moved R20 24.6 mm to (103.4, 108.4), turned to -90 degrees
- moved R19 21.8 mm to (104.9, 108.4), turned to 90 degrees
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
Commit message: All placement done
Parts:
- TP3, TP4, TP5: moved to B.Cu
- moved TP4 36.7 mm to (105.7, 127.9), turned to 90 degrees
- moved C8 31.8 mm to (83.0, 118.1), turned to 180 degrees
- moved TP5 31.7 mm to (102.1, 127.9), turned to 90 degrees
- moved R13 30.1 mm to (104.2, 95.2)
- moved R12 29.7 mm to (102.5, 96.7)
- moved R6 29.3 mm to (104.2, 96.7), turned to 0 degrees
- moved R7 28.5 mm to (102.5, 95.2)
- moved TP3 27.2 mm to (98.8, 127.9), turned to 90 degrees
- moved R18 4.26 mm to (83.8, 114.0), turned to -90 degrees
- moved C15 0.36 mm to (82.8, 116.3)
